File: KiCad_StepperController/KiCad_StepperController.kicad_pcb (KiCad board)
At the start: 2 copper layers, 45 parts, among them J1 Conn_01x01, J2 M1, J3 M1, J4 M1, J5 Conn_01x01, J6 Conn_01x14, SW1 SW_Push, U1 TMC2208, U2 STM32L151RCTx, U3 STLINK-V3MINI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

Commit message: changed formfactor
Parts:
- moved SW1 99.2 mm to (89.0, 129.3), turned to 90 degrees
- moved R4 76.4 mm to (88.9, 120.2)
- moved J6 70.3 mm to (70.2, 99.8)
- moved U2 66.1 mm to (79.7, 116.8)
- moved C27 64.8 mm to (88.9, 113.4)
- moved C28 64.6 mm to (88.9, 115.7)
- moved C26 62.4 mm to (85.9, 127.9), turned to 270 degrees
- moved C23 60.8 mm to (73.6, 124.0), turned to 270 degrees
- moved C22 59.6 mm to (74.0, 109.2), turned to 90 degrees
- moved U3 59.6 mm to (79.7, 130.8)
- moved C21 59.1 mm to (87.0, 111.0)
- moved C25 59.0 mm to (88.9, 117.9)
- moved J1 59.0 mm to (87.0, 99.8)
- moved C6 56.5 mm to (94.4, 103.6)
- moved C24 56.1 mm to (85.9, 123.9), turned to 90 degrees
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Routing:
- net GND: track 15.7 -> 63.6 mm, vias 0 -> 3
- net Net-(J2-Pad4): track 0.00 -> 21.0 mm, vias 0 -> 3
- net Net-(J3-Pad4): track 0.00 -> 20.6 mm, vias 0 -> 3
- net Net-(C1-Pad1): track 0.00 -> 13.1 mm, vias 0 -> 2
- net Net-(J4-Pad2): track 16.0 -> 3.49 mm, vias 3 -> 0
- net Net-(C8-Pad1): track 0.00 -> 12.0 mm, vias 0 -> 2
- net Net-(J4-Pad1): track 15.5 -> 4.84 mm, vias 3 -> 0
- net Net-(J3-Pad3): track 0.00 -> 8.83 mm, vias 0 -> 3
- net Net-(J2-Pad3): track 0.00 -> 8.82 mm, vias 0 -> 3
- net Net-(J4-Pad4): track 29.3 -> 20.9 mm
- net Net-(J4-Pad3): track 16.3 -> 8.84 mm
- net Net-(C11-Pad1): track 0.00 -> 5.10 mm
- net Net-(C3-Pad1): track 0.00 -> 5.09 mm
- net Net-(J2-Pad1): track 0.00 -> 4.82 mm
- net Net-(J3-Pad1): track 0.00 -> 4.82 mm
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- added copper zone on B.Cu, net GND
- removed copper zone on B.Cu, net Net-(J4-Pad1)
- removed copper zone on F.Cu, net Net-(J4-Pad1)
- removed copper zone on B.Cu, net Net-(J4-Pad2)
- removed copper zone on F.Cu, net Net-(J4-Pad2)
- removed copper zone on B.Cu, net Net-(J4-Pad3)
- removed copper zone on F.Cu, net Net-(J4-Pad3)
- removed copper zone on B.Cu, net Net-(J4-Pad4)
- removed copper zone on F.Cu, net Net-(J4-Pad4)
Other:
- board outline added: 47 x 38 mm
